Commit message: ordeno repo, agrego docu y friccion a las patas del perro

File: src/fixed_camera/urdf/fixed_camera.xacro (robot description, xacro)
@@ -1,48 +1,48 @@
 <?xml version="1.0"?>
-<robot xmlns:xacro="http://www.ros.org/wiki/xacro" name="drone_camera">
+<robot xmlns:xacro="http://www.ros.org/wiki/xacro" name="fixed_camera">
     <!-- Properties -->
-    <xacro:property name="drone_body_radius" value="0.15"/>
-    <xacro:property name="drone_body_height" value="0.08"/>
-    <xacro:property name="drone_mass" value="1.5"/>
+    <xacro:property name="body_size" value="0.06"/>
+    <xacro:property name="body_mass" value="0.5"/>
     <xacro:property name="camera_size" value="0.03"/>
     <xacro:property name="camera_mass" value="0.05"/>
     <!-- Materials -->
-    <material name="drone_black">
-        <color rgba="0.1 0.1 0.1 1"/>
+    <material name="body_dark">
+        <color rgba="0.2 0.2 0.2 1"/>
     </material>
     <material name="camera_gray">
         <color rgba="0.5 0.5 0.5 1"/>
     </material>
-    <!-- Base link (center of drone) -->
-    <link name="drone_base_link">
+    <!-- Base link (camera mount body) -->
+    <link name="camera_base_link">
         <inertial>
             <origin xyz="0 0 0" rpy="0 0 0"/>
-            <mass value="${drone_mass}"/>
-            <inertia ixx="0.0082" ixy="0" ixz="0" iyy="0.0082" iyz="0" izz="0.0145"/>
+            <mass value="${body_mass}"/>
+            <inertia ixx="0.0001" ixy="0" ixz="0" iyy="0.0001" iyz="0" izz="0.0001"/>
         </inertial>
         <visual>
             <origin xyz="0 0 0" rpy="0 0 0"/>
             <geometry>
-                <cylinder radius="${drone_body_radius}" length="${drone_body_height}"/>
+                <box size="${body_size} ${body_size} ${body_size}"/>
             </geometry>
-            <material name="drone_black"/>
+            <material name="body_dark"/>
         </visual>
         <collision>
             <origin xyz="0 0 0" rpy="0 0 0"/>
             <geometry>
-                <cylinder radius="${drone_body_radius}" length="${drone_body_height}"/>
+                <box size="${body_size} ${body_size} ${body_size}"/>
             </geometry>
         </collision>
     </link>
-    <!-- Gazebo properties for base link -->
-    <gazebo reference="drone_base_link">
+    <!-- Fixed in the air (no gravity) -->
+    <gazebo reference="camera_base_link">
         <material>Gazebo/DarkGrey</material>
         <gravity>false</gravity>
+        <static>true</static>
     </gazebo>
-    <!-- Camera link -->
+    <!-- Camera link (pointing down) -->
     <joint name="camera_joint" type="fixed">
-        <parent link="drone_base_link"/>
+        <parent link="camera_base_link"/>
         <child link="camera_link"/>
-        <origin xyz="0 0 ${-drone_body_height/2 - camera_size/2}" rpy="0 ${pi/2} 0"/>
+        <origin xyz="0 0 ${-body_size/2 - camera_size/2}" rpy="0 ${pi/2} 0"/>
     </joint>
     <link name="camera_link">
@@ -68,8 +68,8 @@
     <gazebo reference="camera_link">
         <material>Gazebo/Grey</material>
-        <sensor type="camera" name="drone_camera">
+        <sensor type="camera" name="fixed_camera">
             <update_rate>30.0</update_rate>
             <visualize>true</visualize>
-            <camera name="drone_camera">
+            <camera name="fixed_camera">
                 <horizontal_fov>1.396</horizontal_fov>
                 <image>
@@ -98,7 +98,7 @@
             <plugin name="camera_controller" filename="libgazebo_ros_camera.so">
                 <ros>
-                    <namespace>/drone</namespace>
-                    <remapping>~/image_raw:=camera/image_raw</remapping>
-                    <remapping>~/camera_info:=camera/camera_info</remapping>
+                    <namespace>/fixed_camera</namespace>
+                    <remapping>~/image_raw:=image_raw</remapping>
+                    <remapping>~/camera_info:=camera_info</remapping>
                 </ros>
                 <camera_name>camera</camera_name>
@@ -115,26 +115,3 @@
     </joint>
     <link name="camera_link_optical"/>
-    <!-- Propeller markers (visual only) -->
-    <xacro:macro name="propeller" params="name x y">
-        <joint name="${name}_joint" type="fixed">
-            <parent link="drone_base_link"/>
-            <child link="${name}_link"/>
-            <origin xyz="${x} ${y} ${drone_body_height/2 + 0.01}" rpy="0 0 0"/>
-        </joint>
-        <link name="${name}_link">
-            <visual>
-                <geometry>
-                    <cylinder radius="0.08" length="0.005"/>
-                </geometry>
-                <material name="drone_black"/>
-            </visual>
-        </link>
-        <gazebo reference="${name}_link">
-            <material>Gazebo/Black</material>
-        </gazebo>
-    </xacro:macro>
-    <xacro:propeller name="propeller_fl" x="0.10" y="0.10"/>
-    <xacro:propeller name="propeller_fr" x="0.10" y="-0.10"/>
-    <xacro:propeller name="propeller_bl" x="-0.10" y="0.10"/>
-    <xacro:propeller name="propeller_br" x="-0.10" y="-0.10"/>
 </robot>
